Commit message: fix movingtf

File: urdf/simple_pole.urdf.xacro (robot description, xacro)
@@ -10,5 +10,5 @@
 		<link name="${prefix}tool_disk">
 			<visual>
-				<origin xyz="0 0 0" rpy="0 0 0" />
+				<origin xyz="0 0 0.005" rpy="0 0 0" />
 				<geometry>
 					<cylinder length="0.010" radius="0.038"/>
